File: Speakers.sch (KiCad schematic (older format))
At the start: 16 parts, among them J1 SR, J2 SL, J3 SAR, J4 SAL, J5 SBR, J6 SBL, J7 5V, Q1 S8050, Q2 S8050, U1 WeMos_mini

Commit message: Zmiana wartości R1 i R2
Parts:
- R1, R2: value 1k -> 1k8
Changed lines of the file:
@@
 LIBS:valves
 LIBS:relays
-LIBS:ESP8266
-LIBS:wemos_mini
-LIBS:AutoKominek0-cache
-LIBS:Kominek-cache
 LIBS:Speakers-cache
 EELAYER 25 0
@@
 P 9250 3000
 F 0 "R1" V 9330 3000 50  0000 C CNN
-F 1 "1k" V 9250 3000 50  0000 C CNN
+F 1 "1k8" V 9250 3000 50  0000 C CNN
 F 2 "Resistors_SMD:R_1206_HandSoldering" V 9180 3000 50  0001 C CNN
 F 3 "" H 9250 3000 50  0001 C CNN
@@
 P 9250 4250
 F 0 "R2" V 9330 4250 50  0000 C CNN
-F 1 "1k" V 9250 4250 50  0000 C CNN
+F 1 "1k8" V 9250 4250 50  0000 C CNN
 F 2 "Resistors_SMD:R_1206_HandSoldering" V 9180 4250 50  0001 C CNN
 F 3 "" H 9250 4250 50  0001 C CNN
